File: prototypes/clickwheel/AT42QT2120-breakout-v0.sch (EAGLE design)
At the start: 5 parts

Commit message: update ATQ breakouts
Parts:
- removed CLICKWHEEL, DATA: (no value), pinhead:PINHD-1X3/90
- removed RESET: (no value), pinhead:PINHD-1X1
- added CONTROL, JP1: (no value), pinhead:PINHD-1X4/90
Connections:
- removed net N$1: RESET.1, U$1.RESET
- removed net N$2: DATA.1, U$1.CHANGE
- removed net N$4: DATA.2, U$1.SCL
- removed net N$8: DATA.3, U$1.SDA
- new net CHANGE: CONTROL.4, U$1.CHANGE
- new net N$3: JP1.1, U$1.KEY3/GPO1
- new net RESET: CONTROL.2, U$1.RESET
- new net SCL: CONTROL.3, U$1.SCL
- new net SDA: CONTROL.1, U$1.SDA
- net GND: now also U$1.VSS; no longer U$1.VDD
- net N$5: now also JP1.4; no longer CLICKWHEEL.3
- net N$6: now also JP1.3; no longer CLICKWHEEL.2
- net N$7: now also JP1.2; no longer CLICKWHEEL.1
- net V3P3: now also U$1.VDD; no longer U$1.VSS
Changed lines of the file:
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@@
 <?xml version="1.0" encoding="utf-8"?>
 <!DOCTYPE eagle SYSTEM "eagle.dtd">
-<eagle version="9.2.2">
+<eagle version="9.3.0">
 <drawing>
 <settings>
@@
 </classes>
 <parts>
-<part name="DATA" library="pinhead" library_urn="urn:adsk.eagle:library:325" deviceset="PINHD-1X3" device="/90" package3d_urn="urn:adsk.eagle:package:22459/2"/>
 <part name="POWER" library="pinhead" library_urn="urn:adsk.eagle:library:325" deviceset="PINHD-1X2" device="/90" package3d_urn="urn:adsk.eagle:package:22437/2"/>
-<part name="CLICKWHEEL" library="pinhead" library_urn="urn:adsk.eagle:library:325" deviceset="PINHD-1X3" device="/90" package3d_urn="urn:adsk.eagle:package:22459/2"/>
 <part name="U$1" library="AT42QT2120" deviceset="COMMS-AT42QT2120" device="SU" package3d_urn="urn:adsk.eagle:package:30991/2"/>
-<part name="RESET" library="pinhead" library_urn="urn:adsk.eagle:library:325" deviceset="PINHD-1X1" device="" package3d_urn="urn:adsk.eagle:package:22485/2"/>
+<part name="JP1" library="pinhead" library_urn="urn:adsk.eagle:library:325" deviceset="PINHD-1X4" device="/90" package3d_urn="urn:adsk.eagle:package:22404/2"/>
+<part name="CONTROL" library="pinhead" library_urn="urn:adsk.eagle:library:325" deviceset="PINHD-1X4" device="/90" package3d_urn="urn:adsk.eagle:package:22404/2"/>
 </parts>
 <sheets>
@@
 </plain>
 <instances>
-<instance part="DATA" gate="A" x="-38.1" y="-12.7" smashed="yes" rot="MR0">
-<attribute name="NAME" x="-31.75" y="-6.985" size="1.778" layer="95" rot="MR0"/>
-<attribute name="VALUE" x="-31.75" y="-20.32" size="1.778" layer="96" rot="MR0"/>
-</instance>
 <instance part="POWER" gate="G$1" x="-66.04" y="15.24" smashed="yes" rot="R180">
 <attribute name="NAME" x="-59.69" y="9.525" size="1.778" layer="95" rot="R180"/>
 <attribute name="VALUE" x="-59.69" y="20.32" size="1.778" layer="96" rot="R180"/>
 </instance>
-<instance part="CLICKWHEEL" gate="A" x="53.34" y="-22.86" smashed="yes">
-<attribute name="NAME" x="46.99" y="-17.145" size="1.778" layer="95"/>
-<attribute name="VALUE" x="46.99" y="-30.48" size="1.778" layer="96"/>
-</instance>
 <instance part="U$1" gate="G$1" x="0" y="0" smashed="yes">
 <attribute name="NAME" x="-5.08" y="33.02" size="1.778" layer="94"/>
 </instance>
-<instance part="RESET" gate="G$1" x="-66.04" y="27.94" smashed="yes" rot="R180">
-<attribute name="NAME" x="-59.69" y="24.765" size="1.778" layer="95" rot="R180"/>
-<attribute name="VALUE" x="-59.69" y="33.02" size="1.778" layer="96" rot="R180"/>
+<instance part="JP1" gate="A" x="58.42" y="-22.86" smashed="yes">
+<attribute name="NAME" x="52.07" y="-14.605" size="1.778" layer="95"/>
+<attribute name="VALUE" x="52.07" y="-30.48" size="1.778" layer="96"/>
+</instance>
+<instance part="CONTROL" gate="A" x="-58.42" y="-10.16" smashed="yes" rot="R180">
+<attribute name="NAME" x="-52.07" y="-18.415" size="1.778" layer="95" rot="R180"/>
+<attribute name="VALUE" x="-52.07" y="-2.54" size="1.778" layer="96" rot="R180"/>
 </instance>
 </instances>
@@
 <net name="V3P3" class="0">
 <segment>
-<pinref part="U$1" gate="G$1" pin="VSS"/>
-<wire x1="-20.32" y1="17.78" x2="-27.94" y2="17.78" width="0.1524" layer="91"/>
-<label x="-30.48" y="20.32" size="1.778" layer="95"/>
-</segment>
-<segment>
 <pinref part="POWER" gate="G$1" pin="1"/>
 <wire x1="-63.5" y1="12.7" x2="-48.26" y2="12.7" width="0.1524" layer="91"/>
 <label x="-48.26" y="10.16" size="1.778" layer="95"/>
 </segment>
-</net>
-<net name="GND" class="0">
 <segment>
 <pinref part="U$1" gate="G$1" pin="VDD"/>
 <wire x1="-20.32" y1="12.7" x2="-27.94" y2="12.7" width="0.1524" layer="91"/>
-<label x="-30.48" y="10.16" size="1.778" layer="95"/>
-</segment>
+<label x="-33.02" y="10.16" size="1.778" layer="95"/>
+</segment>
+</net>
+<net name="GND" class="0">
 <segment>
 <pinref part="POWER" gate="G$1" pin="2"/>
@@
 <label x="-27.94" y="-33.02" size="1.778" layer="95"/>
 </segment>
-</net>
-<net name="N$2" class="0">
-<segment>
-<pinref part="DATA" gate="A" pin="1"/>
-<wire x1="-35.56" y1="-10.16" x2="-25.4" y2="-10.16" width="0.1524" layer="91"/>
-<wire x1="-25.4" y1="-10.16" x2="-25.4" y2="-7.62" width="0.1524" layer="91"/>
-<pinref part="U$1" gate="G$1" pin="CHANGE"/>
-<wire x1="-25.4" y1="-7.62" x2="-20.32" y2="-7.62" width="0.1524" layer="91"/>
-</segment>
-</net>
-<net name="N$4" class="0">
-<segment>
-<pinref part="DATA" gate="A" pin="2"/>
-<wire x1="-35.56" y1="-12.7" x2="-25.4" y2="-12.7" width="0.1524" layer="91"/>
-<wire x1="-25.4" y1="-12.7" x2="-25.4" y2="-17.78" width="0.1524" layer="91"/>
-<pinref part="U$1" gate="G$1" pin="SCL"/>
-<wire x1="-25.4" y1="-17.78" x2="-20.32" y2="-17.78" width="0.1524" layer="91"/>
+<segment>
+<pinref part="U$1" gate="G$1" pin="VSS"/>
+<wire x1="-20.32" y1="17.78" x2="-27.94" y2="17.78" width="0.1524" layer="91"/>
+<label x="-33.02" y="17.78" size="1.778" layer="95"/>
 </segment>
 </net>
@@
 <wire x1="20.32" y1="-27.94" x2="33.02" y2="-27.94" width="0.1524" layer="91"/>
 <wire x1="33.02" y1="-27.94" x2="33.02" y2="-25.4" width="0.1524" layer="91"/>
-<pinref part="CLICKWHEEL" gate="A" pin="3"/>
-<wire x1="33.02" y1="-25.4" x2="50.8" y2="-25.4" width="0.1524" layer="91"/>
+<wire x1="33.02" y1="-25.4" x2="55.88" y2="-25.4" width="0.1524" layer="91"/>
+<pinref part="JP1" gate="A" pin="4"/>
 </segment>
 </net>
@@
 <segment>
 <pinref part="U$1" gate="G$1" pin="KEY1"/>
-<pinref part="CLICKWHEEL" gate="A" pin="2"/>
-<wire x1="20.32" y1="-22.86" x2="50.8" y2="-22.86" width="0.1524" layer="91"/>
+<wire x1="20.32" y1="-22.86" x2="55.88" y2="-22.86" width="0.1524" layer="91"/>
+<pinref part="JP1" gate="A" pin="3"/>
 </segment>
 </net>
@@
 <wire x1="20.32" y1="-17.78" x2="33.02" y2="-17.78" width="0.1524" layer="91"/>
 <wire x1="33.02" y1="-17.78" x2="33.02" y2="-20.32" width="0.1524" layer="91"/>
-<pinref part="CLICKWHEEL" gate="A" pin="1"/>
-<wire x1="33.02" y1="-20.32" x2="50.8" y2="-20.32" width="0.1524" layer="91"/>
-</segment>
-</net>
-<net name="N$8" class="0">
+<wire x1="33.02" y1="-20.32" x2="55.88" y2="-20.32" width="0.1524" layer="91"/>
+<pinref part="JP1" gate="A" pin="2"/>
+</segment>
+</net>
+<net name="N$3" class="0">
+<segment>
+<pinref part="U$1" gate="G$1" pin="KEY3/GPO1"/>
+<wire x1="20.32" y1="-12.7" x2="35.56" y2="-12.7" width="0.1524" layer="91"/>
+<wire x1="35.56" y1="-12.7" x2="35.56" y2="-17.78" width="0.1524" layer="91"/>
+<pinref part="JP1" gate="A" pin="1"/>
+<wire x1="35.56" y1="-17.78" x2="55.88" y2="-17.78" width="0.1524" layer="91"/>
+</segment>
+</net>
+<net name="RESET" class="0">
+<segment>
+<pinref part="U$1" gate="G$1" pin="RESET"/>
+<wire x1="-20.32" y1="27.94" x2="-27.94" y2="27.94" width="0.1524" layer="91"/>
+<label x="-35.56" y="27.94" size="1.778" layer="95"/>
+</segment>
+<segment>
+<pinref part="CONTROL" gate="A" pin="2"/>
+<wire x1="-55.88" y1="-12.7" x2="-50.8" y2="-12.7" width="0.1524" layer="91"/>
+<label x="-50.8" y="-12.7" size="1.778" layer="95"/>
+</segment>
+</net>
+<net name="SDA" class="0">
+<segment>
+<pinref part="CONTROL" gate="A" pin="1"/>
+<wire x1="-55.88" y1="-15.24" x2="-50.8" y2="-15.24" width="0.1524" layer="91"/>
+<label x="-50.8" y="-15.24" size="1.778" layer="95"/>
+</segment>
 <segment>
 <pinref part="U$1" gate="G$1" pin="SDA"/>
-<wire x1="-20.32" y1="-12.7" x2="-22.86" y2="-12.7" width="0.1524" layer="91"/>
-<wire x1="-22.86" y1="-12.7" x2="-22.86" y2="-15.24" width="0.1524" layer="91"/>
-<pinref part="DATA" gate="A" pin="3"/>
-<wire x1="-22.86" y1="-15.24" x2="-35.56" y2="-15.24" width="0.1524" layer="91"/>
-</segment>
-</net>
-<net name="N$1" class="0">
-<segment>
-<pinref part="RESET" gate="G$1" pin="1"/>
-<pinref part="U$1" gate="G$1" pin="RESET"/>
-<wire x1="-63.5" y1="27.94" x2="-20.32" y2="27.94" width="0.1524" layer="91"/>
-</segment>
-</net>
+<wire x1="-20.32" y1="-12.7" x2="-25.4" y2="-12.7" width="0.1524" layer="91"/>
+<label x="-30.48" y="-12.7" size="1.778" layer="95"/>
+</segment>
+</net>
+<net name="SCL" class="0">
+<segment>
+<pinref part="U$1" gate="G$1" pin="SCL"/>
+<wire x1="-25.4" y1="-17.78" x2="-20.32" y2="-17.78" width="0.1524" layer="91"/>
+<label x="-30.48" y="-17.78" size="1.778" layer="95"/>
+</segment>
+<segment>
+<pinref part="CONTROL" gate="A" pin="3"/>
+<wire x1="-55.88" y1="-10.16" x2="-50.8" y2="-10.16" width="0.1524" layer="91"/>
+<label x="-50.8" y="-10.16" size="1.778" layer="95"/>
+</segment>
+</net>
+<net name="CHANGE" class="0">
+<segment>
+<pinref part="CONTROL" gate="A" pin="4"/>
+<wire x1="-55.88" y1="-7.62" x2="-50.8" y2="-7.62" width="0.1524" layer="91"/>
+<label x="-50.8" y="-7.62" size="1.778" layer="95"/>
+</segment>
+<segment>
+<pinref part="U$1" gate="G$1" pin="CHANGE"/>
+<wire x1="-20.32" y1="-7.62" x2="-25.4" y2="-7.62" width="0.1524" layer="91"/>
+<label x="-35.56" y="-7.62" size="1.778" layer="95"/>
+</segment>
+</net>

Commit message: update ATQ prototype board files
Connections:
- net N$5 renamed KEY0
Changed lines of the file:
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@@
 </segment>
 </net>
-<net name="N$5" class="0">
+<net name="KEY0" class="0">
 <segment>
 <pinref part="U$1" gate="G$1" pin="KEY0"/>
@@
 <wire x1="33.02" y1="-25.4" x2="55.88" y2="-25.4" width="0.1524" layer="91"/>
 <pinref part="JP1" gate="A" pin="4"/>
+<label x="33.02" y="-27.94" size="1.778" layer="95"/>
 </segment>
 </net>
