File: temp/Draft0.brd (EAGLE design)
At the start: 77.5 x 100 mm, 33 parts, among them IC1 REG1117, Q2 MC-306, T1 2N2222, X2 PG203J

Commit message: lab07: pre-checkout? not proud but it's what we sbumitted
Parts:
- removed BATT1: (no value), pinhead:1X02/90
- removed C16, C18, C21: 0.01uF, rcl:C2012
- removed C17, C19: 0.1uF, rcl:C2012
- removed C20: 1uF, rcl:C2012
- removed IC1: REG1117, burr-brown:SOT223
- removed TP9: PTR1PAD1-17, testpad:P1-17
- added ANT1: PRO-OB-440, PRO-OB-440:PRO-OB-440_1
- added C2: .1uF, rcl:C0603
- added C3: 10uF, rcl:C0603
- added C4: 4.7 uF, rcl:C0805
- added C5: 10 uF, rcl:C1210
- added CN1: (no value), adafruit:JST-PH-2-SMT-RA
- added IC2: TPS6300, texas:DRC-S-PVSON-N10
- added R3: 100, rcl:R01005
- added TPS6224: TPS62240, TPS62240:TSP62240
- added U$3: 2.2uH, VLF4012:INDUCTOR
- added U$4: CP2102N-A02-GQFN28, CP2102N-A02-GQFN28:QFN28
- added U$5: CR43NP-2R2MC, CR43NP-4R7MC:INDUCTOR
- added X1: USB-A, adafruit:MOLEX_480371000
- C26: value 10nF -> 47nF
- U$6: value COMMS-AT42QT2120SU -> COMMS-AT42QT2120XU; device AT42QT2120:SO20W -> AT42QT2120:TSSOP20
- moved Q2 76.6 mm to (71.9, 78.0)
- moved C26 66.1 mm to (71.1, 44.3)
- moved C25 61.1 mm to (71.1, 61.2)
- moved U$1 54.6 mm to (34.3, 82.5)
- moved C23 54.4 mm to (71.9, 74.3), turned to 180 degrees
- moved C22 50.5 mm to (66.7, 83.5), turned to 90 degrees
- moved C24 45.5 mm to (61.2, 61.7), turned to 180 degrees
- moved R14 45.2 mm to (63.8, 79.6), turned to 180 degrees
- moved U$7 42.8 mm to (55.9, 82.5)
- moved X2 39.9 mm to (69.8, 53.2), turned to 180 degrees
- moved R13 38.5 mm to (64.3, 74.4)
- moved R1 35.5 mm to (43.3, 83.2), turned to 270 degrees
- moved WHEEL_C 31.1 mm to (74.9, 25.1), turned to 270 degrees
- moved C27 30.5 mm to (49.0, 81.1), turned to 180 degrees
- moved MOT1 30.4 mm to (11.7, 55.7), flipped to the bottom, turned to 180 degrees
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Connections:
- removed net TP7: BATT1.1, IC1.3, TP9.TP
- new net N$10: TPS6224.4, U$5.P$1
- new net N$11: U$4.P$4, X1.3
- new net N$12: U$4.P$5, X1.2
- new net N$3: C2.1, IC2.6, IC2.7, IC2.8, R3.1
- new net N$6: IC2.2, U$3.P$2
- new net N$7: ANT1.2, U$1.2
- new net N$8: IC2.4, U$3.P$1
- new net V1P8: C5.1, TPS6224.5, U$5.P$2, U$7.24, U$7.31, U$7.5, U$7.7
- new net VBAT: C1.1, C3.1, CN1.1, D1.C, IC2.5, MOT1.VCC, R3.2
- new net VBUS: X1.1
- new net VDD: U$4.P$6
- new net VREGIN: U$4.P$7
- net DISPLAY_CS: now also U$1.30; no longer U$1.21
- net GND: now also ANT1.1, C2.2, C3.2, C4.2, C5.2, CN1.2, IC2.3, IC2.9, TPS6224.2, U$4.P$0, U$4.P$3, X1.4; no longer BATT1.2, C16.2, C17.2, C18.2, C19.2, C20.2, C21.2, IC1.1
- net SPI_CLK: now also U$1.31; no longer U$1.17
- net SPI_MISO: now also U$1.32; no longer U$1.18
- net SPI_MOSI: now also U$1.33; no longer U$1.20
- net V3P3: now also C4.1, IC2.1, IC2.10, TPS6224.1, TPS6224.3; no longer C1.1, C16.1, C17.1, C18.1, C19.1, C20.1, C21.1, D1.C, IC1.2, MOT1.VCC, U$7.24, U$7.31, U$7.5, U$7.7
Routing:
- net V3P3: track 0.00 -> 214.9 mm, vias 0 -> 3
- net VBAT: track 0.00 -> 84.2 mm, vias 0 -> 1
- net V1P8: track 0.00 -> 73.1 mm, vias 0 -> 2
- net N$33: track 0.00 -> 65.1 mm, vias 0 -> 3
- net SPI_CLK: track 0.00 -> 59.5 mm, vias 0 -> 2
- net SPI_MOSI: track 0.00 -> 57.7 mm, vias 0 -> 2
- net N$7: track 0.00 -> 55.2 mm
- net N$34: track 0.00 -> 53.5 mm, vias 0 -> 2
- net N$35: track 0.00 -> 47.0 mm, vias 0 -> 2
- net DISPLAY_RST: track 0.00 -> 44.2 mm, vias 0 -> 1
- net VS1053_CS: track 0.00 -> 39.2 mm, vias 0 -> 2
- net DISPLAY_DC: track 0.00 -> 38.0 mm, vias 0 -> 1
- net N$2: track 0.00 -> 37.5 mm, vias 0 -> 2
- net DISPLAY_CS: track 0.00 -> 30.9 mm, vias 0 -> 1
- net VS1053_DREQ: track 0.00 -> 29.4 mm, vias 0 -> 2
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- added copper zone on layer 1, net GND
Other:
- board size 77.5 x 100 mm -> 77.5 x 81 mm

Commit message: updated motor
Parts:
- removed T1: 2N2222, adafruit:TO92-EBC-OVAL
- added Q1: ON_SEMI_MMBT5551LT1GON_SEMI_MMBT5551LT1G_0_0, ON Semi - MMBT5551LT1G:ON_SEMI_MMBT5551LT1G_0
Connections:
- net GND: now also Q1.2, Q1.3; no longer T1.C, T1.E
- net N$2: now also Q1.1; no longer T1.B
Routing:
- net N$2: track 37.5 -> 31.5 mm
