File: temp/Draft0.sch (EAGLE design)
At the start: 33 parts, among them IC1 REG1117, Q2 MC-306, T1 2N2222, X2 PG203J

Commit message: lab07: pre-checkout? not proud but it's what we sbumitted
Parts:
- removed BATT1: (no value), pinhead:PINHD-1X2/90
- removed C16, C18, C21: 0.01uF, rcl:C-EUC2012
- removed C17, C19: 0.1uF, rcl:C-EUC2012
- removed C20: 1uF, rcl:C-EUC2012
- removed IC1: REG1117, burr-brown:REG1117
- removed TP9: PTR1PAD1-17, testpad:PTR1PAD1-17
- added ANT1: PRO-OB-440, PRO-OB-440:PRO-OB-440
- added C2: .1uF, rcl:C-USC0603
- added C3: 10uF, rcl:C-USC0603
- added C4: 4.7 uF, rcl:C-USC0805
- added C5: 10 uF, rcl:C-USC1210
- added CN1: (no value), adafruit:JST_2PIN-SMT-RA
- added IC2: TPS6300, texas:TPS6300
- added R3: 100, rcl:R-US_01005
- added TPS6224: TPS62240, TPS62240:TPS62240
- added U$3: 2.2uH, VLF4012:VLS4012
- added U$4: CP2102N-A02-GQFN28, CP2102N-A02-GQFN28:CP2102N-A02-GQFN28
- added U$5: CR43NP-2R2MC, CR43NP-4R7MC:CR43NP-2R2MC
- added X1: USB-A, adafruit:USB-A
- C26: value 10nF -> 47nF
- U$6: value COMMS-AT42QT2120SU -> COMMS-AT42QT2120XU; device AT42QT2120:COMMS-AT42QT2120SU -> AT42QT2120:COMMS-AT42QT2120XU
Connections:
- removed net TP7: BATT1.1, IC1.VIN, TP9.TP
- new net N$10: TPS6224.SW, U$5.1
- new net N$11: U$4.D+, X1.D+
- new net N$12: U$4.D-, X1.D-
- new net N$3: C2.1, IC2G$1.EN, IC2G$1.PS/SYNC, IC2G$1.VINA, R3.1
- new net N$6: IC2G$1.L2, U$3.2
- new net N$7: ANT1.RF_FEED, U$1.LNA_IN
- new net N$8: IC2G$1.L1, U$3.1
- new net V1P8: C5.1, TPS6224.FB, U$5.2, U$7.CVDD0, U$7.CVDD1, U$7.CVDD2, U$7.CVDD3
- new net VBAT: C1.1, C3.1, CN1.2, D1.C, IC2G$1.VIN, MOT1.VCC, R3.2
- net DISPLAY_CS: now also U$1.SIO3; no longer U$1.IO15
- net GND: now also ANT1.GND, C2.2, C3.2, C4.2, C5.2, CN1.1, IC2G$1.GND, IC2G$1.PGND, TPS6224.GND, U$4.GND_0, U$4.GND_1, X1.GND; no longer BATT1.2, C16.2, C17.2, C18.2, C19.2, C20.2, C21.2, IC1.GND
- net SPI_CLK: now also U$1.SCLK; no longer U$1.IO14
- net SPI_MISO: now also U$1.SIO2; no longer U$1.IO12
- net SPI_MOSI: now also U$1.SIO0; no longer U$1.IO13
- net V3P3: now also C4.1, IC2G$1.FB, IC2G$1.VOUT, TPS6224.EN, TPS6224.VIN; no longer C1.1, C16.1, C17.1, C18.1, C19.1, C20.1, C21.1, D1.C, IC1.VOUT, MOT1.VCC, U$7.CDVDD0, U$7.CVDD1, U$7.CVDD2, U$7.CVDD3
Other:
- note added: "TPS6224"

Commit message: updated motor
Parts:
- removed D1: 1N4004, adafruit:1N4004
- removed T1: 2N2222, adafruit:2N2222
- added D2: ON_SEMI_1N914BWSON_SEMI_1N914BWS_0_0, ON Semi - 1N914BWS:ON_SEMI_1N914BWSON_SEMI_1N914BWS_0_0
- added Q1: ON_SEMI_MMBT5551LT1GON_SEMI_MMBT5551LT1G_0_0, ON Semi - MMBT5551LT1G:ON_SEMI_MMBT5551LT1GON_SEMI_MMBT5551LT1G_0_0
- R1: value 1K -> 1.5K; device adafruit:R-US_R0402 -> adafruit:R-US_R0603
Connections:
- net GND: now also D2.ANODE, Q1.COLLECTOR, Q1.EMITTER; no longer D1.A, T1.C, T1.E
- net N$2: now also Q1.BASE; no longer T1.B
- net VBAT: now also D2.CATHODE; no longer D1.C
Changed lines of the file:
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@@
 <parts>
 <part name="U$1" library="ESP32" deviceset="ESP32-PICO" device="-D4"/>
-<part name="T1" library="adafruit" deviceset="2N2222" device=""/>
-<part name="D1" library="adafruit" deviceset="1N4004" device=""/>
-<part name="R1" library="adafruit" deviceset="R-US_" device="R0402" value="1K"/>
 <part name="C1" library="adafruit" deviceset="C-US" device="025-024X044" value="0.1 uF"/>
 <part name="MOT1" library="Mini-Motor" deviceset="MINI-MOTOR" device=""/>
@@
 <part name="GND4" library="supply1" library_urn="urn:adsk.eagle:library:371" deviceset="GND" device=""/>
 <part name="GND5" library="supply1" library_urn="urn:adsk.eagle:library:371" deviceset="GND" device=""/>
+<part name="Q1" library="ON Semi - MMBT5551LT1G" deviceset="ON_SEMI_MMBT5551LT1G" device="ON_SEMI_MMBT5551LT1G_0_0"/>
+<part name="D2" library="ON Semi - 1N914BWS" deviceset="ON_SEMI_1N914BWS" device="ON_SEMI_1N914BWS_0_0"/>
+<part name="R1" library="adafruit" library_urn="urn:adsk.eagle:library:420" deviceset="R-US_" device="R0603" package3d_urn="urn:adsk.eagle:package:6240565/1" value="1.5K"/>
 </parts>
 <sheets>
@@
 </plain>
 <instances>
-<instance part="T1" gate="G$1" x="10.16" y="25.4" smashed="yes">
-<attribute name="NAME" x="0" y="25.4" size="1.778" layer="95"/>
-<attribute name="VALUE" x="0" y="22.86" size="1.778" layer="96"/>
-</instance>
-<instance part="D1" gate="1" x="5.08" y="40.64" smashed="yes" rot="R90">
-<attribute name="NAME" x="4.5974" y="43.18" size="1.778" layer="95" rot="R90"/>
-<attribute name="VALUE" x="7.3914" y="43.18" size="1.778" layer="96" rot="R90"/>
+<instance part="C1" gate="G$1" x="-5.08" y="43.18" smashed="yes">
+<attribute name="NAME" x="-4.064" y="43.815" size="1.778" layer="95"/>
+<attribute name="VALUE" x="-4.064" y="38.989" size="1.778" layer="96"/>
+</instance>
+<instance part="MOT1" gate="G$1" x="-15.24" y="35.56" smashed="yes" rot="R90"/>
+<instance part="GND20" gate="1" x="-15.24" y="22.86" smashed="yes">
+<attribute name="VALUE" x="-17.78" y="20.32" size="1.778" layer="96"/>
+</instance>
+<instance part="GND21" gate="1" x="12.7" y="12.7" smashed="yes">
+<attribute name="VALUE" x="10.16" y="10.16" size="1.778" layer="96"/>
+</instance>
+<instance part="Q1" gate="G$0" x="7.62" y="33.02" smashed="yes">
+<attribute name="NAME" x="15.24" y="27.94" size="2.54" layer="95" align="top-left"/>
+</instance>
+<instance part="D2" gate="G$0" x="7.62" y="38.1" smashed="yes" rot="R90">
+<attribute name="NAME" x="7.112" y="39.116" size="2.54" layer="95" rot="R90" align="top-left"/>
 </instance>
 <instance part="R1" gate="G$1" x="-2.54" y="15.24" smashed="yes" rot="R90">
 <attribute name="NAME" x="-4.0386" y="11.43" size="1.778" layer="95" rot="R90"/>
 <attribute name="VALUE" x="0.762" y="11.43" size="1.778" layer="96" rot="R90"/>
-</instance>
-<instance part="C1" gate="G$1" x="-5.08" y="43.18" smashed="yes">
-<attribute name="NAME" x="-4.064" y="43.815" size="1.778" layer="95"/>
-<attribute name="VALUE" x="-4.064" y="38.989" size="1.778" layer="96"/>
-</instance>
-<instance part="MOT1" gate="G$1" x="-15.24" y="35.56" smashed="yes" rot="R90"/>
-<instance part="GND20" gate="1" x="-15.24" y="22.86" smashed="yes">
-<attribute name="VALUE" x="-17.78" y="20.32" size="1.778" layer="96"/>
-</instance>
-<instance part="GND21" gate="1" x="12.7" y="12.7" smashed="yes">
-<attribute name="VALUE" x="10.16" y="10.16" size="1.778" layer="96"/>
 </instance>
 </instances>
@@
 <net name="N$2" class="0">
 <segment>
-<pinref part="T1" gate="G$1" pin="B"/>
+<wire x1="-2.54" y1="25.4" x2="-2.54" y2="20.32" width="0.1524" layer="91"/>
+<pinref part="Q1" gate="G$0" pin="BASE"/>
+<wire x1="-2.54" y1="25.4" x2="5.08" y2="25.4" width="0.1524" layer="91"/>
 <pinref part="R1" gate="G$1" pin="2"/>
-<wire x1="7.62" y1="25.4" x2="-2.54" y2="25.4" width="0.1524" layer="91"/>
-<wire x1="-2.54" y1="25.4" x2="-2.54" y2="20.32" width="0.1524" layer="91"/>
 </segment>
 </net>
@@
 <pinref part="C1" gate="G$1" pin="2"/>
 <wire x1="-5.08" y1="35.56" x2="-5.08" y2="38.1" width="0.1524" layer="91"/>
-<pinref part="D1" gate="1" pin="A"/>
-<wire x1="-5.08" y1="35.56" x2="5.08" y2="35.56" width="0.1524" layer="91"/>
-<wire x1="5.08" y1="35.56" x2="5.08" y2="38.1" width="0.1524" layer="91"/>
-<wire x1="5.08" y1="35.56" x2="12.7" y2="35.56" width="0.1524" layer="91"/>
-<junction x="5.08" y="35.56"/>
-<pinref part="T1" gate="G$1" pin="C"/>
-<wire x1="12.7" y1="35.56" x2="12.7" y2="30.48" width="0.1524" layer="91"/>
+<wire x1="-5.08" y1="35.56" x2="12.7" y2="35.56" width="0.1524" layer="91"/>
 <pinref part="MOT1" gate="G$1" pin="GND"/>
 <wire x1="-15.24" y1="30.48" x2="-5.08" y2="30.48" width="0.1524" layer="91"/>
@@
 <wire x1="-15.24" y1="30.48" x2="-15.24" y2="25.4" width="0.1524" layer="91"/>
 <junction x="-15.24" y="30.48"/>
+<pinref part="Q1" gate="G$0" pin="COLLECTOR"/>
+<wire x1="12.7" y1="35.56" x2="12.7" y2="33.02" width="0.1524" layer="91"/>
+<pinref part="D2" gate="G$0" pin="ANODE"/>
+<junction x="12.7" y="35.56"/>
 </segment>
 <segment>
 <pinref part="GND21" gate="1" pin="GND"/>
-<pinref part="T1" gate="G$1" pin="E"/>
-<wire x1="12.7" y1="20.32" x2="12.7" y2="15.24" width="0.1524" layer="91"/>
+<pinref part="Q1" gate="G$0" pin="EMITTER"/>
+<wire x1="12.7" y1="15.24" x2="12.7" y2="17.78" width="0.1524" layer="91"/>
 </segment>
 </net>
 <net name="IO18" class="0">
 <segment>
-<pinref part="R1" gate="G$1" pin="1"/>
 <wire x1="-2.54" y1="10.16" x2="-2.54" y2="7.62" width="0.1524" layer="91"/>
 <wire x1="-2.54" y1="7.62" x2="-12.7" y2="7.62" width="0.1524" layer="91"/>
 <label x="-15.24" y="10.16" size="1.778" layer="95"/>
+<pinref part="R1" gate="G$1" pin="1"/>
 </segment>
 </net>
@@
 <pinref part="C1" gate="G$1" pin="1"/>
 <wire x1="-5.08" y1="45.72" x2="-5.08" y2="50.8" width="0.1524" layer="91"/>
-<wire x1="-5.08" y1="50.8" x2="5.08" y2="50.8" width="0.1524" layer="91"/>
-<pinref part="D1" gate="1" pin="C"/>
-<wire x1="5.08" y1="50.8" x2="5.08" y2="43.18" width="0.1524" layer="91"/>
+<wire x1="-5.08" y1="50.8" x2="12.7" y2="50.8" width="0.1524" layer="91"/>
 <wire x1="-5.08" y1="50.8" x2="-5.08" y2="60.96" width="0.1524" layer="91"/>
 <junction x="-5.08" y="50.8"/>
@@
 <wire x1="-5.08" y1="66.04" x2="0" y2="66.04" width="0.1524" layer="91"/>
 <label x="2.54" y="66.04" size="1.778" layer="95"/>
-</segment>
-</net>
+<pinref part="D2" gate="G$0" pin="CATHODE"/>
+</segment>
+</net>

Commit message: added header for motor
Parts:
- removed MOT1: MINI-MOTOR, Mini-Motor:MINI-MOTOR
- added J1: JST_S3B-XH-SM4-TBJST_S3B-XH-SM4-TB_0_0, JST-S3B-XH-SM4-TB:JST_S3B-XH-SM4-TBJST_S3B-XH-SM4-TB_0_0
Connections:
- net GND: now also J1.2; no longer MOT1.GND
- net VBAT: now also J1.1; no longer MOT1.VCC
Other:
- note removed: "Motor"
Changed lines of the file:
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@@
 <part name="U$1" library="ESP32" deviceset="ESP32-PICO" device="-D4"/>
 <part name="C1" library="adafruit" deviceset="C-US" device="025-024X044" value="0.1 uF"/>
-<part name="MOT1" library="Mini-Motor" deviceset="MINI-MOTOR" device=""/>
 <part name="U$6" library="AT42QT2120" deviceset="COMMS-AT42QT2120" device="XU" package3d_urn="urn:adsk.eagle:package:4349/2" value="COMMS-AT42QT2120XU"/>
 <part name="GND19" library="supply1" library_urn="urn:adsk.eagle:library:371" deviceset="GND" device=""/>
@@
 <part name="D2" library="ON Semi - 1N914BWS" deviceset="ON_SEMI_1N914BWS" device="ON_SEMI_1N914BWS_0_0"/>
 <part name="R1" library="adafruit" library_urn="urn:adsk.eagle:library:420" deviceset="R-US_" device="R0603" package3d_urn="urn:adsk.eagle:package:6240565/1" value="1.5K"/>
+<part name="J1" library="JST-S3B-XH-SM4-TB" deviceset="JST_S3B-XH-SM4-TB" device="JST_S3B-XH-SM4-TB_0_0"/>
 </parts>
 <sheets>
@@
 <description>Vibration Motor</description>
 <plain>
-<text x="-17.78" y="40.64" size="1.778" layer="104" rot="R90">Motor</text>
 </plain>
 <instances>
@@
 <attribute name="VALUE" x="-4.064" y="38.989" size="1.778" layer="96"/>
 </instance>
-<instance part="MOT1" gate="G$1" x="-15.24" y="35.56" smashed="yes" rot="R90"/>
 <instance part="GND20" gate="1" x="-15.24" y="22.86" smashed="yes">
 <attribute name="VALUE" x="-17.78" y="20.32" size="1.778" layer="96"/>
@@
 <attribute name="NAME" x="-4.0386" y="11.43" size="1.778" layer="95" rot="R90"/>
 <attribute name="VALUE" x="0.762" y="11.43" size="1.778" layer="96" rot="R90"/>
+</instance>
+<instance part="J1" gate="G$0" x="-43.18" y="66.04" smashed="yes">
+<attribute name="NAME" x="-40.64" y="63.5" size="2.54" layer="95" align="top-left"/>
 </instance>
 </instances>
@@
 <wire x1="-5.08" y1="35.56" x2="-5.08" y2="38.1" width="0.1524" layer="91"/>
 <wire x1="-5.08" y1="35.56" x2="12.7" y2="35.56" width="0.1524" layer="91"/>
-<pinref part="MOT1" gate="G$1" pin="GND"/>
 <wire x1="-15.24" y1="30.48" x2="-5.08" y2="30.48" width="0.1524" layer="91"/>
 <wire x1="-5.08" y1="30.48" x2="-5.08" y2="35.56" width="0.1524" layer="91"/>
@@
 <pinref part="GND20" gate="1" pin="GND"/>
 <wire x1="-15.24" y1="30.48" x2="-15.24" y2="25.4" width="0.1524" layer="91"/>
-<junction x="-15.24" y="30.48"/>
 <pinref part="Q1" gate="G$0" pin="COLLECTOR"/>
 <wire x1="12.7" y1="35.56" x2="12.7" y2="33.02" width="0.1524" layer="91"/>
 <pinref part="D2" gate="G$0" pin="ANODE"/>
 <junction x="12.7" y="35.56"/>
+<pinref part="J1" gate="G$0" pin="2"/>
+<wire x1="-22.86" y1="50.8" x2="-15.24" y2="50.8" width="0.1524" layer="91"/>
+<wire x1="-15.24" y1="50.8" x2="-15.24" y2="30.48" width="0.1524" layer="91"/>
+<junction x="-15.24" y="30.48"/>
 </segment>
 <segment>
@@
 <junction x="-5.08" y="50.8"/>
 <wire x1="-5.08" y1="60.96" x2="-15.24" y2="60.96" width="0.1524" layer="91"/>
-<pinref part="MOT1" gate="G$1" pin="VCC"/>
-<wire x1="-15.24" y1="60.96" x2="-15.24" y2="58.42" width="0.1524" layer="91"/>
 <wire x1="-5.08" y1="60.96" x2="-5.08" y2="66.04" width="0.1524" layer="91"/>
 <junction x="-5.08" y="60.96"/>
@@
 <label x="2.54" y="66.04" size="1.778" layer="95"/>
 <pinref part="D2" gate="G$0" pin="CATHODE"/>
-</segment>
-</net>
+<pinref part="J1" gate="G$0" pin="1"/>
+<wire x1="-22.86" y1="55.88" x2="-15.24" y2="55.88" width="0.1524" layer="91"/>
+<wire x1="-15.24" y1="55.88" x2="-15.24" y2="60.96" width="0.1524" layer="91"/>
+</segment>
+</net>

Commit message: updated screen
Parts:
- added X3: FH12-45S-0.5SH, con-hirose:FH12-45S-0.5SH
Connections:
- new net N$13: X3-3.1, X3-36.1, X3-37.1, X3-4.1, X3-40.1, X3-5.1
- new net N$14: X3-6.1
- new net N$15: X3-34.1
- new net N$16: X3-32.1
- new net N$17: X3-30.1
- new net N$9: C1.2, D2.ANODE, J1.2, Q1.COLLECTOR
- net GND: now also X3-38.1, X3-39.1, X3-41.1; no longer C1.2, D2.ANODE, J1.2, Q1.COLLECTOR, U$2.GND
- net V3P3: now also U$7.RX
Other:
- moved on the sheet: U$2

Commit message: screen fixes
Parts:
- removed U$2: ADAFRUITST7735R_18, AdafruitST7735R_18:ADAFRUITST7735R_18
Connections:
- net DISPLAY_CS: no longer U$2.TFT_CS
- net DISPLAY_DC: no longer U$2.D/C
- net DISPLAY_RST: no longer U$2.RESET
- net GND: now also X3-10.1, X3-11.1, X3-12.1, X3-13.1, X3-14.1, X3-15.1, X3-16.1, X3-17.1, X3-18.1, X3-19.1, X3-20.1, X3-21.1, X3-22.1, X3-23.1, X3-24.1, X3-25.1, X3-26.1, X3-27.1, X3-28.1, X3-31.1, X3-33.1, X3-7.1, X3-8.1, X3-9.1
- net N$13: now also X3-2.1; no longer X3-3.1
- net SPI_CLK: no longer U$2.SCK
- net SPI_MOSI: no longer U$2.MOSI
- net V3P3: no longer U$2.LITE, U$2.VCC
Other:
- note added: "CLK"
- note added: "CS"
- note added: "MOSI"
- note added: "RST"
- note added: "V3P3"

Commit message: added testpads
Connections:
- net GND: no longer U$7.MICN, U$7.MICP/LINE1
Changed lines of the file:
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@@
 <segment>
 <pinref part="U$7" gate="G$1" pin="DGND0"/>
-<wire x1="-33.02" y1="149.86" x2="-40.64" y2="149.86" width="0.1524" layer="91"/>
-<wire x1="-40.64" y1="149.86" x2="-50.8" y2="149.86" width="0.1524" layer="91"/>
+<wire x1="-33.02" y1="149.86" x2="-50.8" y2="149.86" width="0.1524" layer="91"/>
 <wire x1="-50.8" y1="149.86" x2="-50.8" y2="88.9" width="0.1524" layer="91"/>
 <pinref part="GND25" gate="1" pin="GND"/>
@@
 <wire x1="60.96" y1="27.94" x2="66.04" y2="27.94" width="0.1524" layer="91"/>
 <junction x="66.04" y="27.94"/>
-<pinref part="U$7" gate="G$1" pin="MICP/LINE1"/>
-<wire x1="-33.02" y1="165.1" x2="-40.64" y2="165.1" width="0.1524" layer="91"/>
-<pinref part="U$7" gate="G$1" pin="MICN"/>
-<wire x1="-40.64" y1="165.1" x2="-40.64" y2="160.02" width="0.1524" layer="91"/>
-<wire x1="-40.64" y1="160.02" x2="-33.02" y2="160.02" width="0.1524" layer="91"/>
-<wire x1="-40.64" y1="160.02" x2="-40.64" y2="149.86" width="0.1524" layer="91"/>
-<junction x="-40.64" y="160.02"/>
-<junction x="-40.64" y="149.86"/>
 <pinref part="R13" gate="G$1" pin="2"/>
 <pinref part="C22" gate="G$1" pin="1"/>
