File: hardware/boards/V0/V0.brd (EAGLE design)
At the start: 45 x 104 mm, 149 parts, among them IC2 TPS6300, J12 3.5mm TRRS Jack, J2 HIROSE_DM3BT-DSF-PEJSHIROSE_D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, J3 MOLEX_105450-0101MOLEX_105450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, Q2 ON_SEMI_MMBT5551LT1GON_SEMI_M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, U1 VS1053-L, U2 MICROCHIP_MCP73831T-2ATI-OTMI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, X3 FH12-45S-0.5SH

Commit message: checkpoint
Parts:
- C24, C25: device rcl:C/6032-28R -> rcl:C0402
- C34: device rcl:C1206 -> rcl:C0402
- moved R36 163.2 mm to (-21.7, -45.9), flipped to the bottom
- moved R44 102.9 mm to (8.77, -53.6), flipped to the bottom
- moved C32 71.9 mm to (31.5, -48.0), turned to 0 degrees
- moved R50 62.4 mm to (7.67, -53.3)
- moved C34 51.6 mm to (-7.84, -40.1), turned to 270 degrees
- moved R53 46.8 mm to (3.30, 8.00), flipped to the bottom, turned to 180 degrees
- moved R55 32.2 mm to (-21.1, -48.1), flipped to the bottom, turned to 90 degrees
- moved R25 18.5 mm to (-30.5, -27.5)
- moved D1 15.7 mm to (-21.7, -51.9), turned to 270 degrees
- moved R47 4.04 mm to (6.72, -55.8), turned to 90 degrees
- moved R46 3.27 mm to (5.68, -55.8), turned to 270 degrees
- moved Q1 2.91 mm to (8.49, -58.5), turned to 90 degrees
- moved C40 2.10 mm to (-6.40, -36.5)
- moved C43 2.10 mm to (-6.40, -33.5)
- moved C19 1.80 mm to (-4.12, -37.1)
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Connections:
- net GND: now also C24.2, C25.2; no longer C24.-, C25.-
- net V3P3: now also C24.1, C25.1; no longer C24.+, C25.+
Routing:
- net IO2: track 20.5 -> 52.1 mm, vias 0 -> 2
- net DISPLAY_RST: track 0.00 -> 28.3 mm
- net V3P3: track 220.0 -> 247.2 mm
- net TRRS_INLINE_CTRL: track 0.00 -> 21.3 mm
- net SPI_MISO: track 0.00 -> 16.2 mm
- net SPI_MOSI: track 0.00 -> 15.2 mm
- net BLUE_GREEN_LED_CATH: track 0.00 -> 12.7 mm
- net SPI_CLK: track 0.00 -> 11.3 mm
- net DISPLAY_CS: track 0.00 -> 9.93 mm
- net N$31: track 0.00 -> 9.41 mm, vias 0 -> 1
- net RED_LED_CATH: track 0.00 -> 8.67 mm
- net N$56: track 0.00 -> 7.32 mm
- net RTS: track 2.34 -> 8.16 mm, vias 0 -> 2
- net EN: track 0.00 -> 5.55 mm
- net DTR: track 2.22 -> 6.97 mm
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