File: hardware/boards/Backup/Backup.brd (EAGLE design)
At the start: 100.3 x 100 mm, 25 parts, among them X1 STEREOJACK

Commit message: backup board with fixes
Parts:
- moved VS1053-1 0.32 mm to (74.0, 27.7)
- turned SDCARD to 90 degrees
Connections:
- removed net CARD_DETECT: SDCARD.1
- removed net IO0: ESP32-1.17
- removed net N$29: VS1053-2.6
- removed net N$30: VS1053-2.5, X1.2
- new net N$21: VS1053-2.5, X1.1
- net GND: now also SDCARD.8, VS1053-1.13, VS1053-2.6; no longer SDCARD.3
- net IO12: now also R17.1, SDCARD.3; no longer R14.1, SDCARD.7
- net IO13: now also R16.1, SDCARD.4; no longer R15.1, SDCARD.6
- net IO14: now also R14.1, SDCARD.7; no longer R17.1, SDCARD.4
- net IO15: now also R15.1; no longer R16.1
- net IO2: now also ESP32-1.17, R13.1; no longer R12.1
- net IO4: now also R12.1, SDCARD.10; no longer R13.1, SDCARD.8
- net N$1: no longer VS1053-2.4, X1.5
- net N$13: now also VS1053-2.4, X1.5; no longer VS1053-1.13
- net N$17: now also X1.2; no longer X1.3
- net V3P3: now also SDCARD.6; no longer SDCARD.10, SDCARD.2
Routing:
- net N$1: track 118.8 -> 0.00 mm, vias 4 -> 0
- net N$30: track 114.7 -> 0.00 mm
- net N$21: track 0.00 -> 105.2 mm
- net N$13: track 0.00 -> 89.5 mm
- net IO10: track 106.1 -> 63.3 mm, vias 6 -> 0
- net IO14: track 77.9 -> 101.6 mm, vias 0 -> 2
- net IO12: track 86.2 -> 63.6 mm, vias 6 -> 0
- net IO15: track 77.0 -> 97.7 mm, vias 4 -> 1
- net IO2: track 117.7 -> 137.1 mm, vias 0 -> 1
- net IO4: track 103.7 -> 118.6 mm, vias 4 -> 0
- net V3P3: track 99.2 -> 111.4 mm, vias 2 -> 1
- net DREQ: track 106.3 -> 109.7 mm, vias 2 -> 0
- net DISPLAY_CS: track 88.9 -> 92.2 mm
- net DISPLAY_RST: track 84.8 -> 83.0 mm, vias 4 -> 2
- net IO13: track 81.2 -> 80.0 mm, vias 6 -> 1
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
Commit message: changes to backup
Parts:
- removed R17: 10k, adafruit:0204V
- added C1: 50uF, rcl:E2,5-7
- added C3, C4, C5, C6: 0.5uF, rcl:C025-024X044
- added R18, R4, R5, R6, R7: 10k, rcl:0207/12
- added R2: 100k, rcl:0207/12
- C2: value 50uF -> 0.5uF; device adafruit:C025-024X044 -> rcl:C025-024X044
- R1: value 100k -> 10k; device adafruit:0204V -> rcl:0207/12
- R10, R11, R3, R8, R9: value 330 -> 10k; device adafruit:0204V -> rcl:0207/12
- R12, R13, R14, R15, R16: value 10k -> 330; device adafruit:0204V -> rcl:0207/12
- moved R3 111.7 mm to (-84.0, -21.0)
- moved R12 108.0 mm to (-92.0, 15.0), turned to 0 degrees
- moved R1 92.9 mm to (9.00, 92.0)
- moved C2 84.0 mm to (-56.0, 60.0), turned to 0 degrees
- moved R16 73.1 mm to (-51.0, 65.0), turned to 0 degrees
- moved R10 71.0 mm to (-51.0, 20.0), turned to 0 degrees
- moved R15 67.6 mm to (-51.0, 70.0), turned to 0 degrees
- moved R14 62.7 mm to (-51.0, 75.0), turned to 0 degrees
- moved R11 54.9 mm to (49.0, -6.00)
- moved R9 54.5 mm to (-51.0, 25.0), turned to 0 degrees
- moved R13 21.3 mm to (26.0, 62.8), turned to 0 degrees
- moved R8 16.3 mm to (26.0, 56.0)
- moved DISPLAY 7.00 mm to (93.0, 81.9)
- moved ESP32-2 3.65 mm to (57.3, 29.3)
- moved S3 2.73 mm to (6.98, 19.2)
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Connections:
- new net N$19: R3.1, S1.3
- new net N$22: R8.1, S2.3
- new net N$23: R9.1, S3.3
- new net N$24: R10.1, S4.3
- new net N$25: R11.1, S5.3
- net 3V3: no longer DISPLAY.10, ESP32-2.1, S1.3, S2.3, S3.3, S4.3, S5.3, VS1053-2.10
- net GND: now also C1.-, R12.1, R13.1, R14.1, R15.1, R16.1; no longer C2.2, R1.1, R10.1, R11.1, R3.1, R8.1, R9.1
- net IO10: now also C5.2, R15.2; no longer S4.1
- net IO12: now also R18.1; no longer R17.1
- net IO13: now also R7.1; no longer R16.1
- net IO14: now also R5.1; no longer R14.1
- net IO15: now also R6.1; no longer R15.1
- net IO2: now also R4.1; no longer R13.1
- net IO25: now also C6.2, R16.2; no longer S5.1
- net IO37: now also C3.2, R13.2; no longer S2.1
- net IO38: now also C2.2, R12.2; no longer S1.1
- net IO4: now also R1.1; no longer R12.1
- net N$20: now also R2.2; no longer R1.2
- net SVP: now also C4.2, R14.2; no longer S3.1
- net V3P3: now also C1.+, C3.1, C4.1, C5.1, C6.1, DISPLAY.10, ESP32-2.1, R1.2, R18.2, R2.1, R4.2, R5.2, R6.2, R7.2, S1.1, S2.1, S3.1, S4.1, S5.1, VS1053-2.10; no longer R12.2, R13.2, R14.2, R15.2, R16.2, R17.2
Routing:
- net 3V3: track 243.6 -> 0.00 mm, vias 4 -> 0
- net IO2: track 137.1 -> 0.00 mm, vias 1 -> 0
- net IO4: track 118.6 -> 0.00 mm
- net IO37: track 115.7 -> 0.00 mm, vias 4 -> 0
- net V3P3: track 111.4 -> 0.00 mm, vias 1 -> 0
- net SPI_CLK: track 111.1 -> 0.00 mm, vias 6 -> 0
- net SPI_MOSI: track 110.7 -> 0.00 mm, vias 4 -> 0
- net DREQ: track 109.7 -> 0.00 mm
- net SPI_MISO: track 106.9 -> 0.00 mm, vias 6 -> 0
- net N$21: track 105.2 -> 0.00 mm
- net N$17: track 104.1 -> 0.00 mm, vias 2 -> 0
- net IO14: track 101.6 -> 0.00 mm, vias 2 -> 0
- net VS_CMD_CS: track 101.2 -> 0.00 mm, vias 2 -> 0
- net IO15: track 97.7 -> 0.00 mm, vias 1 -> 0
- net IO38: track 96.5 -> 0.00 mm, vias 6 -> 0
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
Commit message: most routing done
Parts:
- R1, R10, R11, R12, R13, R14, R15, R16, R18, R2, R3, R4, R5, R6, R7, R8, R9: device rcl:0207/12 -> rcl:0207/10
- moved R12 169.4 mm to (66.0, 76.0), turned to 180 degrees
- moved R16 118.1 mm to (66.0, 81.0), turned to 180 degrees
- moved R3 116.7 mm to (30.0, 4.00)
- moved R14 96.1 mm to (45.0, 79.0), turned to 180 degrees
- moved R15 96.1 mm to (45.0, 74.0)
- moved C2 94.4 mm to (20.0, 4.00)
- moved R2 90.2 mm to (21.0, 81.0), turned to 270 degrees
- moved C5 83.7 mm to (20.0, 10.0)
- moved R10 81.9 mm to (30.0, 8.00)
- moved C6 77.8 mm to (21.0, 51.0)
- moved C4 70.1 mm to (14.0, 54.0)
- moved C3 64.0 mm to (6.00, 39.0)
- moved R9 63.3 mm to (8.00, 48.0), turned to 90 degrees
- moved R11 57.0 mm to (28.0, 47.0), turned to 90 degrees
- moved R13 29.1 mm to (45.0, 84.8), turned to 180 degrees
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Connections:
- removed net 3V3: DISPLAY.2, ESP32-1.18
- net V3P3: now also DISPLAY.2, ESP32-1.18
Routing:
- net V3P3: track 0.00 -> 382.4 mm, vias 0 -> 9
- net N$17: track 0.00 -> 157.0 mm, vias 0 -> 4
- net SPI_CLK: track 0.00 -> 151.9 mm, vias 0 -> 4
- net SPI_MISO: track 0.00 -> 150.4 mm, vias 0 -> 5
- net SPI_MOSI: track 0.00 -> 138.4 mm, vias 0 -> 6
- net N$20: track 0.00 -> 131.3 mm, vias 0 -> 5
- net IO4: track 0.00 -> 128.9 mm, vias 0 -> 2
- net N$13: track 0.00 -> 128.3 mm, vias 0 -> 4
- net IO13: track 0.00 -> 128.2 mm, vias 0 -> 2
- net N$21: track 0.00 -> 123.9 mm, vias 0 -> 2
- net IO14: track 0.00 -> 118.9 mm, vias 0 -> 7
- net IO2: track 0.00 -> 113.2 mm, vias 0 -> 5
- net DISPLAY_RST: track 0.00 -> 111.9 mm, vias 0 -> 2
- net IO38: track 0.00 -> 111.3 mm
- net DISPLAY_CS: track 0.00 -> 100.4 mm, vias 0 -> 2
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