File: hardware/boards/Backup/Backup.brd (EAGLE design)
At the start: 100.3 x 100 mm, 35 parts, among them X1 STEREOJACK

Commit message: board closer
Routing:
- net VS_CMD_CS: track 0.00 -> 93.7 mm, vias 0 -> 1
- net IO37: track 77.4 -> 163.7 mm, vias 4 -> 6
- net IO15: track 59.7 -> 133.3 mm, vias 0 -> 3
- net IO10: track 67.7 -> 108.6 mm, vias 2 -> 3
- net IO13: track 128.2 -> 147.0 mm, vias 2 -> 4
- net IO12: track 93.0 -> 105.4 mm, vias 4 -> 6
- net SPI_MOSI: track 138.4 -> 141.3 mm
- net N$13: track 128.3 -> 127.2 mm
