File: hardware/boards/Backup/Backup.sch (EAGLE design)
At the start: 25 parts, among them X1 STEREOJACK

Commit message: backup board with fixes
Connections:
- removed net CARD_DETECT: SDCARD.1
- removed net IO0: ESP32-1.17
- removed net N$29: VS1053-2.6
- removed net N$30: VS1053-2.5, X1.2
- new net N$21: VS1053-2.5, X1.1
- net GND: now also SDCARD.8, VS1053-1.13, VS1053-2.6; no longer SDCARD.3
- net IO12: now also R17.1, SDCARD.3; no longer R14.1, SDCARD.7
- net IO13: now also R16.1, SDCARD.4; no longer R15.1, SDCARD.6
- net IO14: now also R14.1, SDCARD.7; no longer R17.1, SDCARD.4
- net IO15: now also R15.1; no longer R16.1
- net IO2: now also ESP32-1.17, R13.1; no longer R12.1
- net IO4: now also R12.1, SDCARD.10; no longer R13.1, SDCARD.8
- net N$1: no longer VS1053-2.4, X1.5
- net N$13: now also VS1053-2.4, X1.5; no longer VS1053-1.13
- net N$17: now also X1.2; no longer X1.3
- net V3P3: now also SDCARD.6; no longer SDCARD.10, SDCARD.2
Other:
- note added: "1: DAT2"
- note added: "2: CD/DAT3"
- note added: "3: CMD"
- note added: "4: VDD"
- note added: "5: CLK"
- note added: "6: VSS"
- note added: "7: DAT0"
- note added: "8: DAT1"
- note added: "Card Detect A"
- note added: "Card Detect B"
- moved on the sheet: R12, R13, R14, R15, R16, R17

Commit message: changes to backup
Parts:
- removed R17: 10k, adafruit:R-US_0204/2V
- added C1: 50uF, rcl:CPOL-USE2.5-7
- added C3, C4, C5, C6: 0.5uF, rcl:C-US025-024X044
- added R18, R4, R5, R6, R7: 10k, rcl:R-US_0207/12
- added R2: 100k, rcl:R-US_0207/12
- C2: value 50uF -> 0.5uF; device adafruit:C-US025-024X044 -> rcl:C-US025-024X044
- R1: value 100k -> 10k; device adafruit:R-US_0204/2V -> rcl:R-US_0207/12
- R10, R11, R3, R8, R9: value 330 -> 10k; device adafruit:R-US_0204/2V -> rcl:R-US_0207/12
- R12, R13, R14, R15, R16: value 10k -> 330; device adafruit:R-US_0204/2V -> rcl:R-US_0207/12
Connections:
- new net N$19: R3.1, S1.P
- new net N$22: R8.1, S2.P
- new net N$23: R9.1, S3.P
- new net N$24: R10.1, S4.P
- new net N$25: R11.1, S5.P
- net 3V3: no longer DISPLAY.10, ESP32-2.1, S1.P, S2.P, S3.P, S4.P, S5.P, VS1053-2.10
- net GND: now also C1.-, R12.1, R13.1, R14.1, R15.1, R16.1; no longer C2.2, R1.1, R10.1, R11.1, R3.1, R8.1, R9.1
- net IO10: now also C5.2, R15.2; no longer S4.S
- net IO12: now also R18.1; no longer R17.1
- net IO13: now also R7.1; no longer R16.1
- net IO14: now also R5.1; no longer R14.1
- net IO15: now also R6.1; no longer R15.1
- net IO2: now also R4.1; no longer R13.1
- net IO25: now also C6.2, R16.2; no longer S5.S
- net IO37: now also C3.2, R13.2; no longer S2.S
- net IO38: now also C2.2, R12.2; no longer S1.S
- net IO4: now also R1.1; no longer R12.1
- net N$20: now also R2.2; no longer R1.2
- net SVP: now also C4.2, R14.2; no longer S3.S
- net V3P3: now also C1.+, C3.1, C4.1, C5.1, C6.1, DISPLAY.10, ESP32-2.1, R1.2, R18.2, R2.1, R4.2, R5.2, R6.2, R7.2, S1.S, S2.S, S3.S, S4.S, S5.S, VS1053-2.10; no longer R12.2, R13.2, R14.2, R15.2, R16.2, R17.2

Commit message: most routing done
Parts:
- R1, R10, R11, R12, R13, R14, R15, R16, R18, R2, R3, R4, R5, R6, R7, R8, R9: device rcl:R-US_0207/12 -> rcl:R-US_0207/10
Connections:
- removed net 3V3: DISPLAY.2, ESP32-1.18
- net V3P3: now also DISPLAY.2, ESP32-1.18
