File: hardware/boards/pico/revA/pico.brd (EAGLE design)
At the start: 45 x 104 mm, 149 parts, among them IC2 TPS6300, J12 3.5mm TRRS Jack, J2 HIROSE_DM3BT-DSF-PEJSHIROSE_D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, J3 MOLEX_105450-0101MOLEX_105450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, Q2 ON_SEMI_MMBT5551LT1GON_SEMI_M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, U1 VS1053-L, U2 MICROCHIP_MCP73831T-2ATI-OTMI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, X3 FH12-45S-0.5SH

Commit message: housekeeping + checkpoint
Parts:
- added JP1: (no value), adafruit:1X08-LOCK
- added R56: 0Ω, rcl:R1206
- C1: value 50uF -> 50μF
- C13: value 0.1 uF -> 0.1μF
- C14, C6, C7: value 1uF -> 1μF
- C2: value .1uF -> 0.1μF
- C21, C23, C25, C33, C34, C38: value 0.1uF -> 0.1μF
- C22, C24, C26, C27: value 4.7uF -> 4.7μF
- C28, C29, C3, C32, C37, C4, C43: value 10uF -> 10μF
- C5: value 10 uF -> 10μF
- R1, R2, R26, R32, R4, R40, R41, R42, R43, R48, R49, R5, R50, R53, R6, R7: value 10k -> 10kΩ
- R10, R17, R18, R9: value 100k -> 100kΩ
- R11: value 10M -> 10MΩ
- R12: value 1M -> 1MΩ
- R13: value 10 -> 10Ω
- R14, R15: value 20 -> 20Ω
- R16: value 100K -> 100KΩ
- R19: value 155k -> 155kΩ
- R20: value 75k -> 75kΩ
- R21: value 35k -> 35kΩ
- R22: value 15k -> 15kΩ
- R23, R25, R33: value 5k -> 5kΩ
- R24, R45: value 50k -> 50kΩ
- R27, R28: value 5.1k -> 5.1kΩ
- R29: value 22.1k -> 22.1kΩ
- R3, R35: value 100 -> 100Ω
- R30: value 47.5k -> 47.5kΩ
- R31, R46, R47: value 1k -> 1kΩ
- R34: value 2k -> 2kΩ
- R36: value 50 -> 50Ω
- R37, R38, R39: value 4.7k -> 4.7kΩ
- R44: value 10K -> 10kΩ
- R51: value 180k -> 180kΩ
- R52: value 360k -> 360kΩ
- R54: value 315k -> 315kΩ
- R55: value 25 -> 25Ω
- R8: value 1.5K -> 1.5KΩ
- moved C24 151.8 mm to (-55.9, -7.30), turned to 180 degrees
- moved C25 143.3 mm to (-51.0, 2.10), turned to 180 degrees
- moved R32 129.7 mm to (-48.4, 9.20), turned to 180 degrees
- moved R33 123.8 mm to (-53.9, 12.7), turned to 180 degrees
- moved TP1 88.7 mm to (12.3, -3.20), flipped to the bottom, turned to 0 degrees
- moved R35 77.5 mm to (-53.9, 45.7), turned to 180 degrees
- moved C30 71.6 mm to (-42.7, 20.8)
- moved C31 71.6 mm to (-38.7, 20.8)
- moved R45 71.6 mm to (-57.7, 21.8)
- moved U$7 71.6 mm to (-34.7, 20.8)
- moved R19 50.9 mm to (-24.4, -41.6), flipped to the bottom
- moved C33 49.4 mm to (36.6, -28.9)
- moved ANT1 33.7 mm to (46.5, 4.70)
- moved TP3 0.39 mm to (10.5, -54.1)
- moved R18 0.32 mm to (-3.60, -39.5), turned to 270 degrees
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Connections:
- removed net N$38: R16.2, U1.10, U1.11, U1.12, U1.25, U1.33, U1.34, U1.36, U1.9
- new net N$45: R16.1, U1.10, U1.11, U1.12, U1.25, U1.33, U1.34, U1.36, U1.9
- net DREQ: now also JP1.1
- net GND: now also JP1.7, R16.2; no longer R16.1, R18.1
- net N$41: now also R18.1; no longer R18.2
- net SPI_CLK: now also JP1.4
- net SPI_MISO: now also JP1.6
- net SPI_MOSI: now also JP1.5
- net SYS_ENABLE: now also R56.2
- net V3P3: now also JP1.8, R18.2
- net VBAT: now also R56.1
- net VS_CMD_CS: now also JP1.3
- net VS_DATA_CS: now also JP1.2
Routing:
- net N$45: track 0.00 -> 24.7 mm, vias 0 -> 2
- net N$38: track 24.7 -> 0.00 mm, vias 3 -> 0
- net V3P3: track 247.2 -> 258.0 mm, vias 17 -> 18
- net N$11: track 3.93 -> 5.84 mm
- net V1P8: track 48.5 -> 48.7 mm, vias 0 -> 2

Commit message: checkpoint: pico is trudging along
Parts:
- C30, C31: device rcl:C0201 -> rcl:C0402
- R56: device rcl:R1206 -> rcl:R0603
- moved R56 120.3 mm to (14.2, -14.0), flipped to the bottom, turned to 90 degrees
- moved R45 109.3 mm to (20.4, -54.7), flipped to the bottom, turned to 270 degrees
- moved D1 91.0 mm to (16.9, 30.5), turned to 0 degrees
- moved R55 85.8 mm to (17.9, 28.3), turned to 270 degrees
- moved R36 83.0 mm to (15.5, 28.3), turned to 270 degrees
- moved R35 72.7 mm to (16.7, 28.3), flipped to the bottom, turned to 270 degrees
- moved D7 64.9 mm to (-5.00, -48.5), flipped to the bottom
- moved R21 64.2 mm to (-6.30, -44.5), turned to 270 degrees
- moved R54 62.5 mm to (-11.5, -44.5), flipped to the bottom, turned to 270 degrees
- moved D5 61.3 mm to (-6.30, -51.5), flipped to the bottom
- moved D6 60.6 mm to (-7.60, -48.5), flipped to the bottom
- moved R20 58.9 mm to (-8.90, -44.5), flipped to the bottom, turned to 270 degrees
- moved R33 57.4 mm to (3.30, 7.70), flipped to the bottom
- moved R23 57.4 mm to (-5.00, -44.5), flipped to the bottom, turned to 270 degrees
- moved C30 57.2 mm to (-2.00, -19.4), flipped to the bottom, turned to 0 degrees
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Connections:
- net CENTER_SW_PWR_TOP: now also CENTER_SW_PWR.1, CENTER_SW_PWR.1-2
- net GND: now also CENTER_SW_PWR.3, CENTER_SW_PWR.3-2
- net N$29: now also CENTER_SW.3, CENTER_SW.3-2
- net V3P3: now also CENTER_SW.1, CENTER_SW.1-2
Routing:
- net V3P3: track 258.0 -> 313.0 mm, vias 18 -> 21
- net CENTER_SW_PWR_TOP: track 3.06 -> 53.4 mm, vias 0 -> 1
- net RXD0: track 0.00 -> 44.4 mm, vias 0 -> 2
- net TXD0: track 0.00 -> 42.2 mm, vias 0 -> 2
- net N$28: track 0.00 -> 40.0 mm, vias 0 -> 3
- net N$24: track 4.25 -> 42.3 mm, vias 0 -> 1
- net TRRS_INLINE_CTRL: track 21.3 -> 53.9 mm
- net EN: track 5.55 -> 37.9 mm, vias 0 -> 2
- net DREQ: track 0.00 -> 30.9 mm, vias 0 -> 2
- net SPI_CLK: track 11.3 -> 41.6 mm, vias 0 -> 2
- net VS_CMD_CS: track 0.00 -> 30.2 mm, vias 0 -> 2
- net SPI_MISO: track 16.2 -> 45.4 mm, vias 0 -> 2
- net SPI_MOSI: track 15.2 -> 43.9 mm, vias 0 -> 2
- net RED_LED_CATH: track 8.67 -> 30.6 mm
- net N$16: track 4.25 -> 25.5 mm, vias 0 -> 3
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
Commit message: checkpoint: mostly route complete (!)
Routing:
- net BLUE_GREEN_LED_CATH: track 3.60 -> 96.2 mm, vias 2 -> 4
- net VBAT_ADC_IN: track 1.24 -> 69.9 mm, vias 0 -> 2
- net CHARGE_DETECT: track 0.00 -> 68.7 mm, vias 0 -> 2
- net VIB_MOTOR: track 0.00 -> 54.6 mm, vias 0 -> 2
- net TRRS_TIP_SW: track 3.70 -> 42.1 mm, vias 0 -> 2
- net ATQ_CHANGE: track 11.0 -> 48.9 mm, vias 0 -> 4
- net DISPLAY_CS: track 24.0 -> 60.2 mm, vias 1 -> 2
- net DREQ: track 30.9 -> 66.0 mm, vias 2 -> 4
- net VS_DATA_CS: track 0.00 -> 31.4 mm, vias 0 -> 2
- net DISPLAY_RST: track 40.5 -> 71.9 mm, vias 1 -> 2
- net VS_CMD_CS: track 30.2 -> 60.8 mm, vias 2 -> 4
- net I2C_SCL: track 10.4 -> 40.0 mm, vias 0 -> 2
- net I2C_SDA: track 7.25 -> 36.1 mm, vias 0 -> 2
- net SPI_CLK: track 41.6 -> 66.6 mm, vias 2 -> 4
- net SPI_MOSI: track 43.9 -> 67.6 mm, vias 2 -> 4
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
Commit message: checkpoint: route complete (!!)
Parts:
- moved C25 74.2 mm to (-5.30, -56.4), flipped to the bottom, turned to 270 degrees
- moved C24 71.4 mm to (-4.00, -56.4), flipped to the bottom, turned to 270 degrees
- moved C33 45.6 mm to (-8.42, -36.5), turned to 0 degrees
- moved C32 37.9 mm to (-8.42, -35.4)
- moved C34 0.35 mm to (-8.70, -39.2)
Routing:
- net V3P3: track 313.0 -> 414.3 mm, vias 21 -> 29
- net ATQ_CHANGE: track 48.9 -> 47.5 mm
- net VBAT: track 56.5 -> 57.1 mm
