File: hardware/boards/pico/revA/pico.brd (EAGLE design)
At the start: 45 x 104 mm, 151 parts, among them IC2 TPS6300, J12 3.5mm TRRS Jack, J2 HIROSE_DM3BT-DSF-PEJSHIROSE_D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, J3 MOLEX_105450-0101MOLEX_105450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, Q2 ON_SEMI_MMBT5551LT1GON_SEMI_M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, U1 VS1053-L, U2 MICROCHIP_MCP73831T-2ATI-OTMI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, X3 FH12-45S-0.5SH

Commit message: checkpoint: labels
Parts:
- moved BATT_CON 2.10 mm to (15.4, 16.9), turned to 180 degrees
- moved C2 2.00 mm to (19.7, 6.65)
- moved C3 1.30 mm to (18.3, 3.44)
- moved R3 1.00 mm to (18.4, 4.60)
- renumbered J2 to MICRO_SD, U$7 to L3, X3 to DISPLAY_CONN
Connections:
- net GND: now also BATT_CON.1; no longer BATT_CON.3
- net VBAT: now also BATT_CON.3; no longer BATT_CON.1
Routing:
- net N$3: track 7.06 -> 8.43 mm
- net SPI_CLK: track 66.6 -> 67.7 mm
- net I2C_SDA: track 36.1 -> 37.2 mm
- net VBAT: track 57.1 -> 57.9 mm
- net V3P3: track 414.3 -> 413.7 mm

Commit message: checkpoint: drc, round 2
Routing:
- net VBAT: track 57.9 -> 61.0 mm
- net N$6: track 1.50 -> 4.42 mm
- net V1P8: track 49.2 -> 48.6 mm
Changed lines of the file:
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@@
 <element name="U$3" library="VLF4012" package="INDUCTOR" value="2.2uH" x="10.99" y="0.87" smashed="yes" rot="MR270"/>
 <element name="C2" library="rcl" library_urn="urn:adsk.eagle:library:334" package="C0402" package3d_urn="urn:adsk.eagle:package:23626/2" value="0.1μF" x="19.7" y="6.65" smashed="yes" rot="MR90">
-<attribute name="NAME" x="19.615" y="7.965" size="0.254" layer="26" rot="MR180"/>
+<attribute name="NAME" x="19.615" y="8.065" size="0.254" layer="26" rot="MR180"/>
 <attribute name="SPICEPREFIX" value="C" x="36.7" y="-19.35" size="1.778" layer="28" rot="MR90" display="off"/>
 <attribute name="VALUE" x="19.395" y="5.505" size="0.254" layer="28" rot="MR180"/>
@@
 </element>
 <element name="C19" library="rcl" library_urn="urn:adsk.eagle:library:334" package="C0402" package3d_urn="urn:adsk.eagle:package:23626/2" value="100nF" x="-4.12" y="-37.15" smashed="yes" rot="MR0">
-<attribute name="NAME" x="-3.195" y="-36.59" size="0.4" layer="26" rot="MR0"/>
+<attribute name="NAME" x="-3.495" y="-36.59" size="0.4" layer="26" rot="MR0"/>
 <attribute name="SPICEPREFIX" value="C" x="27.88" y="-98.15" size="1.778" layer="28" rot="MR0" display="off"/>
 <attribute name="VALUE" x="-4.355" y="-36.58" size="0.254" layer="28" rot="MR0"/>
@@
 </element>
 <element name="CH1" library="testpad" library_urn="urn:adsk.eagle:library:385" package="TP20SQ" package3d_urn="urn:adsk.eagle:package:27980/1" value="TPSQTP20SQ" x="10" y="-31" smashed="yes" rot="R180">
-<attribute name="NAME" x="10.5" y="-32.15" size="0.4" layer="25" rot="R180"/>
+<attribute name="NAME" x="10.4" y="-32.15" size="0.4" layer="25" rot="R180"/>
 <attribute name="TP_SIGNAL_NAME" value="" x="10" y="-31" size="1.778" layer="27" rot="R180" display="off"/>
 <attribute name="VALUE" x="11.016" y="-29.857" size="0.0254" layer="27" rot="R180"/>
@@
 <element name="U$4" library="Crystal" package="ECSCRYSTAL" value="ECS12P88MHZ" x="2" y="-26.8" smashed="yes" rot="MR0"/>
 <element name="C30" library="rcl" library_urn="urn:adsk.eagle:library:334" package="C0402" package3d_urn="urn:adsk.eagle:package:23626/2" value="2.7pF" x="-2" y="-19.4" smashed="yes" rot="MR0">
-<attribute name="NAME" x="-1.065" y="-18.865" size="0.4" layer="26" rot="MR0"/>
+<attribute name="NAME" x="-1.265" y="-18.765" size="0.4" layer="26" rot="MR0"/>
 <attribute name="SPICEPREFIX" value="C" x="-2" y="-19.4" size="1.778" layer="28" rot="MR0" display="off"/>
-<attribute name="VALUE" x="-2.265" y="-18.805" size="0.254" layer="28" rot="MR0"/>
+<attribute name="VALUE" x="-2.465" y="-18.705" size="0.254" layer="28" rot="MR0"/>
 </element>
 <element name="C31" library="rcl" library_urn="urn:adsk.eagle:library:334" package="C0402" package3d_urn="urn:adsk.eagle:package:23626/2" value="4.7pF" x="-2.03" y="-22.56" smashed="yes" rot="MR0">
@@
 <wire x1="4.73" y1="4.5" x2="4.99" y2="4.76" width="0.3048" layer="16"/>
 <wire x1="19.95" y1="-11.075" x2="21.5" y2="-9.525" width="0.254" layer="16"/>
-<wire x1="21.5" y1="8.5" x2="20.5" y2="9.5" width="0.3048" layer="16"/>
-<wire x1="20.5" y1="9.5" x2="20" y2="9.5" width="0.3048" layer="16"/>
+<wire x1="20.5" y1="9.5" x2="21.5" y2="8.5" width="0.3048" layer="16"/>
 <wire x1="21.5" y1="-9.525" x2="21.5" y2="-7.5" width="0.3048" layer="16"/>
 <wire x1="21.5" y1="-7.5" x2="21.5" y2="-1.8" width="0.3048" layer="16"/>
@@
 <wire x1="14.881953125" y1="2.4" x2="14.885" y2="2.396953125" width="0.254" layer="16"/>
 <wire x1="14.885" y1="2.396953125" x2="14.885" y2="1.86" width="0.254" layer="16"/>
+<wire x1="17.9" y1="11.85" x2="20.25" y2="9.5" width="0.254" layer="16"/>
+<wire x1="20.25" y1="9.5" x2="20.5" y2="9.5" width="0.254" layer="16"/>
 </signal>
 <signal name="V3P3">
@@
 <wire x1="12.59" y1="-41.2" x2="12.435" y2="-41.355" width="0.4064" layer="16"/>
 <wire x1="12.435" y1="-41.355" x2="12.435" y2="-42.065" width="0.4064" layer="16"/>
-<wire x1="13.02" y1="-42.65" x2="13.02" y2="-42.66" width="0.4064" layer="16"/>
 <wire x1="13.02" y1="-42.65" x2="13.02" y2="-42.63" width="0.4064" layer="16"/>
 <wire x1="12.695" y1="-42.305" x2="13.02" y2="-42.63" width="0.4064" layer="16"/>
@@
 <wire x1="12.72" y1="-43.5" x2="13" y2="-43.5" width="0.4064" layer="16"/>
 <wire x1="12.685" y1="-42.315" x2="12.5" y2="-42.5" width="0.4064" layer="16"/>
-<wire x1="12.5" y1="-42.5" x2="12.5" y2="-42.69" width="0.4064" layer="16"/>
-<wire x1="12.5" y1="-42.69" x2="12.5" y2="-43" width="0.4064" layer="16"/>
+<wire x1="12.5" y1="-42.5" x2="12.5" y2="-43" width="0.4064" layer="16"/>
 <wire x1="12.5" y1="-43" x2="12.5" y2="-43.5" width="0.4064" layer="16"/>
 <wire x1="13" y1="-43.5" x2="13.5" y2="-43" width="0.4064" layer="16"/>
@@
 <wire x1="13" y1="-43" x2="13" y2="-42.63" width="0.4064" layer="16"/>
 <wire x1="12.435" y1="-43" x2="12.5" y2="-43" width="0.4064" layer="16"/>
-<wire x1="13.02" y1="-42.63" x2="12.96" y2="-42.69" width="0.4064" layer="16"/>
-<wire x1="12.96" y1="-42.69" x2="12.5" y2="-42.69" width="0.4064" layer="16"/>
 <wire x1="12.325" y1="-43.325" x2="12.505" y2="-43.325" width="0.4064" layer="16"/>
 <wire x1="12.505" y1="-43.325" x2="12.83" y2="-43" width="0.4064" layer="16"/>
@@
 <contactref element="IC2" pad="2"/>
 <contactref element="U$3" pad="P$2"/>
-<wire x1="10.79" y1="-0.37" x2="10.79" y2="-0.43" width="0.4064" layer="16"/>
-<wire x1="14.885" y1="0.36" x2="13.95" y2="0.36" width="0.4064" layer="16"/>
+<wire x1="13.95" y1="0.36" x2="14.885" y2="0.36" width="0.4064" layer="16"/>
 <polygon width="0.254" layer="16" thermals="no">
 <vertex x="14.011921875" y="0.609059375"/>
@@
 <vertex x="13.5" y="-1.45"/>
 </polygon>
-<wire x1="13.95" y1="0.36" x2="13.45" y2="0.36" width="0.2" layer="16"/>
+<wire x1="10.79" y1="-0.43" x2="11.58" y2="0.36" width="0.254" layer="16"/>
+<wire x1="11.58" y1="0.36" x2="13.95" y2="0.36" width="0.254" layer="16"/>
 </signal>
 <signal name="N$8">
@@
 <wire x1="-2.94225" y1="-20.67775" x2="-2.731125" y2="-20.888875" width="0.2" layer="1" curve="-90"/>
 <wire x1="-2.731125" y1="-20.888875" x2="-2.52" y2="-21.1" width="0.2" layer="1" curve="90"/>
-<wire x1="-2.52" y1="-21.1" x2="5.6" y2="-21.1" width="0.2" layer="1"/>
-<via x="5.6" y="-21.1" extent="1-16" drill="0.25"/>
+<wire x1="-2.52" y1="-21.1" x2="5.9" y2="-21.1" width="0.2" layer="1"/>
+<via x="5.9" y="-21.1" extent="1-16" drill="0.25"/>
 <wire x1="9.94" y1="-21.1" x2="10.03" y2="-21.01" width="0.2" layer="16"/>
-<wire x1="5.6" y1="-21.1" x2="9.94" y2="-21.1" width="0.2" layer="16"/>
+<wire x1="5.9" y1="-21.1" x2="9.94" y2="-21.1" width="0.2" layer="16"/>
 </signal>
 <signal name="I2C_SCL">
@@
 <mfgpreviewcolor name="substratecolor" color="0xFF786E46"/>
 </mfgpreviewcolors>
+<errors>
+</errors>
 </board>
 </drawing>

Commit message: checkpoint: names and such
Routing:
- net N$13: track 0.00 -> 8.87 mm
- net N$47: track 0.00 -> 2.00 mm
- net N$15: track 0.00 -> 2.00 mm
Other:
- board text added: "(rev A)"
- board text added: "Rahul Butani, Blake Martini, Sameer Mithani, Sneha Pendharkar"
Changed lines of the file:
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@@
 <layer number="28" name="bValues" color="7" fill="1" visible="yes" active="yes"/>
 <layer number="29" name="tStop" color="7" fill="3" visible="no" active="yes"/>
-<layer number="30" name="bStop" color="7" fill="6" visible="no" active="yes"/>
+<layer number="30" name="bStop" color="7" fill="6" visible="yes" active="yes"/>
 <layer number="31" name="tCream" color="7" fill="4" visible="no" active="yes"/>
 <layer number="32" name="bCream" color="7" fill="5" visible="no" active="yes"/>
@@
 </polygon>
 <rectangle x1="-21.5" y1="-8.2" x2="8.3" y2="29.8" layer="48"/>
+<text x="-9.4" y="21" size="2.54" layer="16" font="fixed" rot="MR0">(rev A)</text>
+<circle x="-7.4" y="22" radius="1" width="0.4064" layer="30"/>
+<circle x="-7.4" y="22" radius="1" width="0.4064" layer="16"/>
+<wire x1="-0.7" y1="21" x2="-0.7" y2="22.9" width="0.4064" layer="30"/>
+<wire x1="-0.7" y1="22.9" x2="-0.7" y2="23.6" width="0.4064" layer="30"/>
+<wire x1="-0.7" y1="25" x2="-0.7" y2="23.6" width="0.4064" layer="30"/>
+<wire x1="-0.7" y1="22.9" x2="-1.7" y2="22.9" width="0.4064" layer="30"/>
+<wire x1="-1.7" y1="22.9" x2="-2.7" y2="23.9" width="0.4064" layer="30" curve="-90"/>
+<wire x1="-2.7" y1="23.9" x2="-1.6" y2="25" width="0.4064" layer="30" curve="-90"/>
+<wire x1="-1.6" y1="25" x2="-0.7" y2="25" width="0.4064" layer="30"/>
+<wire x1="-3.4" y1="23" x2="-3.4" y2="21" width="0.4064" layer="30"/>
+<wire x1="-3.4" y1="24" x2="-3.4" y2="23.9" width="0.4064" layer="30"/>
+<wire x1="-5.7" y1="23" x2="-5.7" y2="21" width="0.4064" layer="30" curve="-210"/>
+<text x="-0.4" y="9.6" size="1.7" layer="22" font="vector" rot="MR0">Rahul Butani,
+Blake Martini,
+Sameer Mithani,
+Sneha Pendharkar</text>
 </plain>
 <attributes>
@@
 <wire x1="5.04" y1="-33.76" x2="-1.74" y2="-33.76" width="0.2" layer="16"/>
 </signal>
+<signal name="N$13">
+<wire x1="-0.7" y1="21" x2="-0.7" y2="22.9" width="0.4064" layer="16"/>
+<wire x1="-0.7" y1="22.9" x2="-0.7" y2="23.6" width="0.4064" layer="16"/>
+<wire x1="-0.7" y1="25" x2="-0.7" y2="23.6" width="0.4064" layer="16"/>
+<wire x1="-0.7" y1="22.9" x2="-1.7" y2="22.9" width="0.4064" layer="16"/>
+<wire x1="-1.7" y1="22.9" x2="-2.7" y2="23.9" width="0.4064" layer="16" curve="-90"/>
+<wire x1="-2.7" y1="23.9" x2="-1.6" y2="25" width="0.4064" layer="16" curve="-90"/>
+<wire x1="-1.6" y1="25" x2="-0.7" y2="25" width="0.4064" layer="16"/>
+</signal>
+<signal name="N$15">
+<wire x1="-3.4" y1="23" x2="-3.4" y2="21" width="0.4064" layer="16"/>
+</signal>
+<signal name="N$44">
+<wire x1="-3.4" y1="24" x2="-3.4" y2="23.9" width="0.4064" layer="16"/>
+</signal>
+<signal name="N$47">
+<wire x1="-5.7" y1="23" x2="-5.7" y2="21" width="0.4064" layer="16" curve="-210"/>
+</signal>
 </signals>
 <mfgpreviewcolors>
@@
 </drawing>
 <compatibility>
+<note version="6.3" minversion="6.2.2" severity="warning">
+Since Version 6.2.2 text objects can contain more than one line,
+which will not be processed correctly with this version.
+</note>
 <note version="8.2" severity="warning">
 Since Version 8.2, EAGLE supports online libraries. The ids
