File: hardware/boards/pico/revA/wheel.brd (EAGLE design)
At the start: 38 x 38 mm, 0 parts

Commit message: pico: checkpoint: an outdated wheel
Routing:
- net CH1: track 459.1 -> 0.00 mm
- net CH0: track 459.1 -> 0.00 mm
- net CH2: track 459.1 -> 473.8 mm, vias 0 -> 1
- added copper zone on layer 1, net CH0
- added copper zone on layer 16, net CH0
- added copper zone on layer 1, net CH1
- added copper zone on layer 16, net CH1
- added copper zone on layer 1, net CH2
- added copper zone on layer 16, net CH2
- added copper zone on layer 16, net GUARD

Commit message: pico: wheel board, basically complete
Routing:
- net CH2: track 473.8 -> 7.00 mm
- net CH1: track 0.00 -> 11.1 mm, vias 0 -> 1
- net CH0: track 0.00 -> 8.91 mm, vias 0 -> 1
- net GUARD: track 0.00 -> 2.93 mm, vias 0 -> 1
- added copper zone on layer 1, net CH3
- added copper zone on layer 1, net GUARD

Commit message: pico: DON'T PANIC
(yes, I know - it should've been a dolphin or a mouse. gotta save something for revision B. and it's a cute fish.)
Routing:
- net GUARD: track 2.93 -> 2.07 mm
- removed copper zone on layer 16, net GUARD
Other:
- board text added: "CH0"
- board text added: "CH1"
- board text added: "CH2"
- board text added: "DON'T"
- board text added: "GUARD"
- board text added: "PANIC"
